File: schematics/BNO080Connect.kicad_sch (KiCad schematic)
At the start: 1 part, among them J3 Conn_01x10 IMU BNO080

Commit message: Added Footprints
Parts:
- J3: footprint (none) -> Connector_PinSocket_1.00mm:PinSocket_1x10_P1.00mm_Vertical
Changed lines of the file:
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@@
 			)
 		)
-		(property "Footprint" ""
+		(property "Footprint" "Connector_PinSocket_1.00mm:PinSocket_1x10_P1.00mm_Vertical"
 			(at 148.59 92.71 0)
 			(effects
