File: schematics/CANBusModule.kicad_sch (KiCad schematic)
At the start: 7 parts, among them U1 MCP2562-E-MF, U4 MCP2515-xSO, Y2 Crystal

Commit message: Added Footprints
Parts:
- C4, C5, C6: footprint (none) -> Capacitor_SMD:C_0603_1608Metric
- R4: footprint (none) -> Resistor_SMD:R_0603_1608Metric
- Y2: footprint (none) -> Crystal:Crystal_HC49-U-3Pin_Vertical
Changed lines of the file:
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@@
 			)
 		)
-		(property "Footprint" ""
+		(property "Footprint" "Capacitor_SMD:C_0603_1608Metric"
 			(at 155.9052 104.14 0)
 			(effects
@@
 			)
 		)
-		(property "Footprint" ""
+		(property "Footprint" "Resistor_SMD:R_0603_1608Metric"
 			(at 102.362 97.79 90)
 			(effects
@@
 			)
 		)
-		(property "Footprint" ""
+		(property "Footprint" "Capacitor_SMD:C_0603_1608Metric"
 			(at 155.9052 114.3 0)
 			(effects
@@
 			)
 		)
-		(property "Footprint" ""
+		(property "Footprint" "Capacitor_SMD:C_0603_1608Metric"
 			(at 94.9452 106.68 0)
 			(effects
@@
 			)
 		)
-		(property "Footprint" ""
+		(property "Footprint" "Crystal:Crystal_HC49-U-3Pin_Vertical"
 			(at 162.56 105.41 0)
 			(effects
